Commit message: chore: rotate rover model to be right side up

File: rover_2024_description/urdf/Core.xacro (robot description, xacro)
@@ -6,4 +6,11 @@
 <xacro:include filename="$(find rover_2024_description)/urdf/ball_joint.xacro" />
 <link name="base_link">
+</link>
+<joint name="chassis_joint" type="fixed">
+  <parent link="base_link"/>
+  <child link="chassis"/>
+  <origin xyz="0 0 0.3" rpy="${pi/2} 0 0"/>
+</joint>
+<link name="chassis">
   <inertial>
     <origin xyz="-0.01226587986232331 0.09909397702738384 -0.005243928985965616" rpy="0 0 0"/>
@@ -385,4 +392,5 @@
   </collision>
 </link>
+<!-- Joints -->
 <joint name="Revolute 3" type="continuous">
   <origin xyz="0.0001 -0.08972 -0.184859" rpy="0 0 0"/>
@@ -459,5 +467,5 @@
 <xacro:ball_joint
   name="Ball 18"
-  parent="base_link"
+  parent="chassis"
   child="DiffBar2_1"
 >
@@ -466,5 +474,5 @@
 <xacro:ball_joint
   name="Ball 19"
-  parent="base_link"
+  parent="chassis"
   child="DiffBar1_1"
 >
@@ -493,10 +501,10 @@
 <joint name="Planar 27" type="planar">
   <origin xyz="0.027224 0.0 -0.072776" rpy="0 0 0"/>
-  <parent link="base_link"/>
+  <parent link="chassis"/>
   <child link="Diff_1"/>
 </joint>
 <joint name="Revolute 28" type="continuous">
   <origin xyz="-0.2446 0.079599 0.049591" rpy="0 0 0"/>
-  <parent link="base_link"/>
+  <parent link="chassis"/>
   <child link="Rocker1_1"/>
   <axis xyz="-1.0 0.0 0.0"/>
@@ -504,5 +512,5 @@
 <joint name="Revolute 29" type="continuous">
   <origin xyz="0.2476 0.079599 0.049591" rpy="0 0 0"/>
-  <parent link="base_link"/>
+  <parent link="chassis"/>
   <child link="Rocker2_1"/>
   <axis xyz="1.0 0.0 0.0"/>

File: rover_2024_description/urdf/ball_joint.xacro (robot description, xacro)
@@ -3,5 +3,5 @@
 <xacro:macro name="ball_joint" params="name parent child *origin">
   <joint name="${name}_joint" type="continuous">
-    <parent link="base_link"/>
+    <parent link="${parent}"/>
     <child link="${name}_link1"/>
     <axis xyz="0 1 0" />
